File: hardware/fan-characterization-fixture/fan-characterization-fixture.kicad_sch (KiCad schematic)
At the start: 36 parts, among them J1 MCU_IF, J2 BENCH_PSU, J3 FAN_DUT, Q1 NTR4003NT1G

Commit message: fixture: move the Rev 0 controller overlay from N8R8 to N16R8
The fixture still described its controller wiring as an N8R8 breakout
overlay, with reasoning about a CH343P board and the ESP32-S3-DevKitC-1.
The provisional Rev 0 controller is now the N16R8 on Lonely Binary's
carrier, as PR #8's docs/TARGET_N16R8.md records: GPIO6 gate,
CONFIG_DB_FAN_GATE_SINK_LEVEL=1, GPIO7 tach, PPR 0 (unknown). The J1
mapping and sdkconfig lines are unchanged; only the board they belong
to and the reasoning about it change.

The README overlay table, the BRINGUP flash step and the sheet note now
name the N16R8, and the README gives its build overlay chain. The
DevKitC/CH343P paragraph is replaced by what Lonely Binary's map shows
for GPIO6/7, and GPIO48 joins the reserved-pin list. The claims that
GPIO6 has no pull at reset and that its power-up glitch is low were
never checked against the ESP32-S3 datasheet here, so both are now
marked unverified, in the README and on the sheet.

A validation boundary states what the N16R8 has shown (baseline
validated, fan-characterization image booted, static GPIO6 levels with
nothing attached) and what it has not (fixture, external stage, tach
path, 25 kHz waveform; PPR unknown). The pins remain DragonBench
bench-fixture assignments, not JumpJet GPIOs. The schematic, PDF and SVG
are regenerated for the note text only.
Other:
- note added: "Controller-agnostic link. Board wiring is a LOCAL overlay. N16R8 Rev 0 bench overlay (provisional, NOT JumpJet GPIOs): J1.1 MCU_PWM <- GPIO6 J1.2 TACH_GPIO -> GPIO7 J1.3 3V3 <- board 3V3 (never 5V) J1.4 GND <- board GND sdkconfig.fan-characterization.local: CONFIG_DB_FAN_PWM_GATE_GPIO=6 CONFIG_DB_FAN_GATE_SINK_LEVEL=1 CONFIG_DB_FAN_TACH_GPIO=7 TinyS3[D]: same J1 functions, own overlay. Controller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"
- note removed: "Controller-agnostic link. Board wiring is a LOCAL overlay. N8R8 bench overlay (provisional, NOT product GPIOs): J1.1 MCU_PWM <- GPIO6 J1.2 TACH_GPIO -> GPIO7 J1.3 3V3 <- board 3V3 (never 5V) J1.4 GND <- board GND sdkconfig.fan-characterization.local: CONFIG_DB_FAN_PWM_GATE_GPIO=6 CONFIG_DB_FAN_GATE_SINK_LEVEL=1 CONFIG_DB_FAN_TACH_GPIO=7 TinyS3[D]: same J1 functions, own overlay. Breakout is passi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"
Changed lines of the file:
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@@
 )
   (text
-    "Controller-agnostic link. Board wiring is a LOCAL overlay.\nN8R8 bench overlay (provisional, NOT product GPIOs):\n  J1.1 MCU_PWM   <- GPIO6\n  J1.2 TACH_GPIO -> GPIO7\n  J1.3 3V3       <- board 3V3 (never 5V)\n  J1.4 GND       <- board GND\nsdkconfig.fan-characterization.local:\n  CONFIG_DB_FAN_PWM_GATE_GPIO=6\n  CONFIG_DB_FAN_GATE_SINK_LEVEL=1\n  CONFIG_DB_FAN_TACH_GPIO=7\nTinyS3[D]: same J1 functions, own overlay.\nBreakout is passive: no protection assumed."
+    "Controller-agnostic link. Board wiring is a LOCAL overlay.\nN16R8 Rev 0 bench overlay (provisional, NOT JumpJet GPIOs):\n  J1.1 MCU_PWM   <- GPIO6\n  J1.2 TACH_GPIO -> GPIO7\n  J1.3 3V3       <- board 3V3 (never 5V)\n  J1.4 GND       <- board GND\nsdkconfig.fan-characterization.local:\n  CONFIG_DB_FAN_PWM_GATE_GPIO=6\n  CONFIG_DB_FAN_GATE_SINK_LEVEL=1\n  CONFIG_DB_FAN_TACH_GPIO=7\nTinyS3[D]: same J1 functions, own overlay.\nController terminals are passive: no protection assumed."
     (at 19.05 78.74 0)
     (effects (font (size 1.27 1.27)) (justify left top))
 )
   (text
-    "Q1 non-inverting: gate HIGH = sink => CONFIG_DB_FAN_GATE_SINK_LEVEL=1. sink_duty_pct = Q1 on-time.\nFan control input, 9GA0424P3J001 drawing Rev C: 25 kHz specified; open-collector/open-drain drive OK;\n   control open = same speed as 100 %; 0 % = stopped; open voltage <= 5.25 V; source <= 2 mA at 0 V; VIL <= 0.4 V.\nQ1 NTR4003NT1G is a signal-interface FET here: normal stress VDS <= 5.25 V, ID <= 2 mA.\n   Low level at 2 mA: 2 mA x 2.0 ohm (RDS(on) max, VGS 2.5 V) = 4 mV, << 0.4 V.\nR1 220R: gate charge current <= 3.3/220 = 15 mA peak; RC < 25 ns even at 100 pF, vs 20 us half-period.\n   Driven gate = VOH x 10k/10.22k = 3.23 V at 3.3 V (2.94 V at a 3.0 V rail): above the 2.5 V RDS(on) row.\nR2 10k: GPIO Hi-Z/reset/unpowered -> gate = IGSS x 10k (<= 0.1 V at 10 uA, assumed). GPIO6: no pull at reset.\nNOT rated for FAN_PWM_RAW landed on FAN_24V: verify lead identity before landing (BRINGUP step 2).\nNo RC filter and no fixture pull-up on FAN_PWM_RAW. JP2 open = line fully released for open-line tests."
+    "Q1 non-inverting: gate HIGH = sink => CONFIG_DB_FAN_GATE_SINK_LEVEL=1. sink_duty_pct = Q1 on-time.\nFan control input, 9GA0424P3J001 drawing Rev C: 25 kHz specified; open-collector/open-drain drive OK;\n   control open = same speed as 100 %; 0 % = stopped; open voltage <= 5.25 V; source <= 2 mA at 0 V; VIL <= 0.4 V.\nQ1 NTR4003NT1G is a signal-interface FET here: normal stress VDS <= 5.25 V, ID <= 2 mA.\n   Low level at 2 mA: 2 mA x 2.0 ohm (RDS(on) max, VGS 2.5 V) = 4 mV, << 0.4 V.\nR1 220R: gate charge current <= 3.3/220 = 15 mA peak; RC < 25 ns even at 100 pF, vs 20 us half-period.\n   Driven gate = VOH x 10k/10.22k = 3.23 V at 3.3 V (2.94 V at a 3.0 V rail): above the 2.5 V RDS(on) row.\nR2 10k: GPIO Hi-Z/reset/unpowered -> gate = IGSS x 10k (<= 0.1 V at 10 uA, assumed). GPIO6 reset pull: unverified.\nNOT rated for FAN_PWM_RAW landed on FAN_24V: verify lead identity before landing (BRINGUP step 2).\nNo RC filter and no fixture pull-up on FAN_PWM_RAW. JP2 open = line fully released for open-line tests."
     (at 116.84 86.36 0)
     (effects (font (size 1.27 1.27)) (justify left top))
